Commit message: fix(sim): correct right-hand finger mirroring, fix fill-light placement
The mirroring transform in generate_hand.py flipped joint position/rpy per
side but left the z-axis driver joints' rotation axis hardcoded to (0,0,1)
for both hands. Under a y-mirror, rotation sense about a z-axis reverses
(R_z(theta) -> R_z(-theta)) while rotation about a y-axis does not, so
thumb1/ring1/pinky1_joint (axis z) picked up a handedness error on the
right hand that index1/middle1_joint (axis y) never had. It was largest on
ring1/pinky1_joint because their rpy tilt (0.7 rad) mixes much more of the
mis-handled component in than thumb1_joint's small 0.1 rad tilt, which is
why only ring/pinky visibly curled backward. Fixed by flipping axis to
(0,0,-flip) for these three driver joints, regenerated right/hand.urdf +
right/hand.sdf; left hand (already correct) is untouched.

Also in hand_world.sdf:
- fill_light_left/right were placed at y=-0.6, behind the backdrop_wall
  (y=-0.45) instead of in front on the camera's side (y=+0.5) - moved to
  y=+0.6 so they actually reach the hands instead of being blocked by the
  wall.
- Re-enabled cast_shadows on the sun (previously fully disabled due to
  shadow acne on the hand's small close-packed meshes), but kept it off
  specifically on the 36 finger-segment visuals - the documented acne
  source - while leaving it on for hand_link/forearm_link and the
  workbench/backdrop, so there's now a real shadow without the jitter
  regression.
- Darkened ground_plane material to match backdrop_wall's tone.

Also adds sim/worlds/gui/{left_hand,right_hand}.config, the per-side
camera-preset launch profiles referenced in CLAUDE.md but not yet
committed.

Files: 6 changed

File: sim/models/hand/right/hand.urdf (robot description, URDF)
Before this commit: robot inmoov_right_hand, 20 links, 19 joints
Joints:
- joint pinky1_joint: axis 0.000000 0.000000 1.000000 -> 0.000000 0.000000 -1.000000
- joint ring1_joint: axis 0.000000 0.000000 1.000000 -> 0.000000 0.000000 -1.000000
- joint thumb1_joint: axis 0.000000 0.000000 1.000000 -> 0.000000 0.000000 -1.000000
