Commit message: fix(vision,sim): per-finger curl calibration and thumb driver axis
Vision: curl_fraction/angle_to_servo now take an optional finger name and
look up per-finger (straight, curled) overrides via FINGER_CALIBRATION,
falling back to the old shared defaults. The thumb's real curled angle
(measured ~108-109 deg) was nowhere near the shared curled=40 floor, so a
fully curled thumb only ever reported ~50% curled. Added --log-finger to
print a finger's raw angle plus running min/max for calibrating others.

Sim: thumb1_joint's rotation axis was inherited from its original role as
a passive mimic of thumb_joint (multiplier 0.75) in the source xacro, not
from being a driver joint - promoting it to driver (required by
bullet-featherstone's downstream-mimic constraint) kept an axis that was
never meant to reproduce the thumb's actual flexion. Fixed by re-deriving
the axis via rotation composition: thumb_joint's own axis (0,1,0) rotated
through thumb_joint's own rpy, expressed in thumb1_joint's frame. Verified
against direct gz topic pub commands, isolated from vision and physics
gain tuning.

File: sim/models/hand/left/hand.urdf (robot description, URDF)
Before this commit: robot inmoov_left_hand, 20 links, 19 joints
Joints:
- joint thumb1_joint: axis 0.000000 0.000000 1.000000 -> 0.270584 0.626579 -0.730878

File: sim/models/hand/right/hand.urdf (robot description, URDF)
Before this commit: robot inmoov_right_hand, 20 links, 19 joints
Joints:
- joint thumb1_joint: axis 0.000000 0.000000 -1.000000 -> -0.270584 0.626579 0.730878
